File: TARA_LORA8X-S2/TARA_LORA8X-S2.kicad_sch (KiCad schematic)
At the start: 58 parts, among them J11 Screw_Terminal_01x12, J31 Screw_Terminal_01x12, J61 Conn_01x04, K11 HRS1H-S-DC3V, K12 HRS1H-S-DC3V, K13 HRS1H-S-DC3V, K14 HRS1H-S-DC3V, K15 HRS1H-S-DC3V, K16 HRS1H-S-DC3V, K17 HRS2H-S-DC3V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

Commit message: 202504101905
GreenSave windowsๅ11 kicad9.0
Other:
- note added: "TARA_LORA"
