File: 8X8_I2C_Extension/31 I2C_Extension.kicad_sch (KiCad schematic)
At the start: 68 parts, among them J1 Screw_Terminal_01x10, J2 Screw_Terminal_01x12, Q1 2N5401, Q2 2N5401, Q3 2N5401, Q4 2N5401, Q5 2N5401, Q6 2N5401, Q7 2N5401, Q8 2N5401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

Commit message: add I/O identifi
Other:
- note added: "+5V"
- note added: "COM"
- note added: "GND"
- note added: "P1"
- note added: "P2"
- note added: "P3"
- note added: "P4"
- note added: "P5"
- note added: "P6"
- note added: "P7"
- note added: "P8"
- note added: "SCL"
- note added: "SDA"
- note added: "SEN1"
- note added: "SEN2"
- note added: "SEN3"
- note added: "SEN4"
- note added: "SEN5"
- note added: "SEN6"
- note added: "SEN7"
- note added: "SEN8"
- note added: "VCC"
Changed lines of the file:
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@@
     (stroke (width 0) (type default) (color 0 0 0 0))
+  )
+  (text "VCC" (at 18.288 48.514 0)
+    (effects (font (size 1.27 1.27)) (justify left bottom))
+  )
+  (text "P6" (at 18.288 40.894 0)
+    (effects (font (size 1.27 1.27)) (justify left bottom))
+  )
+  (text "P5" (at 18.288 38.354 0)
+    (effects (font (size 1.27 1.27)) (justify left bottom))
+  )
+  (text "SEN5" (at 278.638 37.846 0)
+    (effects (font (size 1.27 1.27)) (justify left bottom))
+  )
+  (text "P4" (at 18.288 35.56 0)
+    (effects (font (size 1.27 1.27)) (justify left bottom))
+  )
+  (text "SDA" (at 278.638 53.086 0)
+    (effects (font (size 1.27 1.27)) (justify left bottom))
+  )
+  (text "P7" (at 18.288 43.434 0)
+    (effects (font (size 1.27 1.27)) (justify left bottom))
+  )
+  (text "SEN3" (at 278.638 32.512 0)
+    (effects (font (size 1.27 1.27)) (justify left bottom))
+  )
+  (text "COM" (at 278.638 48.006 0)
+    (effects (font (size 1.27 1.27)) (justify left bottom))
+  )
+  (text "+5V" (at 278.638 50.546 0)
+    (effects (font (size 1.27 1.27)) (justify left bottom))
+  )
+  (text "GND" (at 18.288 51.054 0)
+    (effects (font (size 1.27 1.27)) (justify left bottom))
+  )
+  (text "P2" (at 18.288 30.734 0)
+    (effects (font (size 1.27 1.27)) (justify left bottom))
+  )
+  (text "SEN6" (at 278.638 40.386 0)
+    (effects (font (size 1.27 1.27)) (justify left bottom))
+  )
+  (text "SEN4" (at 278.638 35.052 0)
+    (effects (font (size 1.27 1.27)) (justify left bottom))
+  )
+  (text "SCL" (at 278.638 55.626 0)
+    (effects (font (size 1.27 1.27)) (justify left bottom))
+  )
+  (text "P3" (at 18.288 33.02 0)
+    (effects (font (size 1.27 1.27)) (justify left bottom))
+  )
+  (text "P8" (at 18.288 45.974 0)
+    (effects (font (size 1.27 1.27)) (justify left bottom))
+  )
+  (text "SEN8" (at 278.638 45.466 0)
+    (effects (font (size 1.27 1.27)) (justify left bottom))
+  )
+  (text "P1" (at 18.288 28.194 0)
+    (effects (font (size 1.27 1.27)) (justify left bottom))
+  )
+  (text "SEN1" (at 278.638 27.686 0)
+    (effects (font (size 1.27 1.27)) (justify left bottom))
+  )
+  (text "SEN7" (at 278.638 42.926 0)
+    (effects (font (size 1.27 1.27)) (justify left bottom))
+  )
+  (text "SEN2" (at 278.638 30.226 0)
+    (effects (font (size 1.27 1.27)) (justify left bottom))
   )
   (label "VCC1" (at 69.85 123.19 0)
