File: 8X8_I2C_Extension/31 I2C_Extension.kicad_pcb (KiCad board)
At the start: 2 copper layers, 122.5 x 87.9 mm, 68 parts, among them J1 Screw_Terminal_01x10, J2 Screw_Terminal_01x12, Q1 2N5401, Q2 2N5401, Q3 2N5401, Q4 2N5401, Q5 2N5401, Q6 2N5401, Q7 2N5401, Q8 2N5401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

Commit message: add versions screen on pcb 8x8 i2c
Other:
- board text added: "V1.0.0"
Changed lines of the file:
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@@
   (gr_arc (start 123.496189 88.346385) (mid 123.273012 88.885209) (end 122.734189 89.108385) (layer "Edge.Cuts") (width 0.2))
   (gr_circle (center 119.699004 85.1818) (end 121.399004 85.1818) (layer "Edge.Cuts") (width 0.1) (fill none))
+  (gr_text "V1.0.0" (at 95 87) (layer "F.SilkS")
+    (effects (font (size 1.5 1.5) (thickness 0.3)))
+  )
   (segment (start 35.06939 34.50939) (end 35.80401 35.24401) (width 0.5) (layer "B.Cu") (net 1))
   (segment (start 23.35401 26.61201) (end 23.35401 34.50939) (width 0.5) (layer "B.Cu") (net 1))

Commit message: 20251006_grennsave_win10_kicad9
Routing:
- net Net-(J2-Pad10): track 71.7 -> 71.0 mm
