File: TARA_T8X/TARA_T8X.kicad_pcb (KiCad board)
At the start: 2 copper layers, 122.5 x 87.9 mm, 137 parts, among them J1 Screw_Terminal_01x10, J2 ESP32-WROOM-32U, J3 Conn_01x04_MountingPin, J4 Screw_Terminal_01x10, Q1 2N5401, Q10 2N5401, Q2 2N5401, Q3 2N5401, Q4 2N5401, Q5 2N5401, Q6 2N5401, Q7 2N5401, Q8 2N5401, Q9 2N5401, U1 CN3903, U2 LM1117-3.3, U3 TTL_RS485_Module, U4 DS1307+, Y1 Crystal_Small

Commit message: 202510061930_greensave
Parts:
- moved R19 1.39 mm to (171.9, 100.3)
- moved R20 1.39 mm to (179.2, 100.3)
- moved R17 1.29 mm to (157.1, 100.3)
- moved R18 1.24 mm to (164.6, 100.3)
- moved R16 1.16 mm to (149.8, 100.2)
Changed lines of the file:
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@@
 	(footprint "Resistor_SMD:R_0805_2012Metric"
 		(layer "F.Cu")
-		(at 157.1 101.5625 90)
+		(at 157.1 100.275 90)
 		(descr "Resistor SMD 0805 (2012 Metric), square (rectangular) end terminal, IPC-7351 nominal, (Body size source: IPC-SM-782 page 72, https://www.pcb-3d.com/wordpress/wp-content/uploads/ipc-sm-782a_amendment_1_and_2.pdf), generated with kicad-footprint-generator")
 		(tags "resistor")
@@
 	(footprint "Resistor_SMD:R_0805_2012Metric"
 		(layer "F.Cu")
-		(at 179.2 101.6625 90)
+		(at 179.2 100.275 90)
 		(descr "Resistor SMD 0805 (2012 Metric), square (rectangular) end terminal, IPC-7351 nominal, (Body size source: IPC-SM-782 page 72, https://www.pcb-3d.com/wordpress/wp-content/uploads/ipc-sm-782a_amendment_1_and_2.pdf), generated with kicad-footprint-generator")
 		(tags "resistor")
@@
 	(footprint "Resistor_SMD:R_0805_2012Metric"
 		(layer "F.Cu")
-		(at 164.6 101.5125 90)
+		(at 164.575 100.275 90)
 		(descr "Resistor SMD 0805 (2012 Metric), square (rectangular) end terminal, IPC-7351 nominal, (Body size source: IPC-SM-782 page 72, https://www.pcb-3d.com/wordpress/wp-content/uploads/ipc-sm-782a_amendment_1_and_2.pdf), generated with kicad-footprint-generator")
 		(tags "resistor")
@@
 	(footprint "Resistor_SMD:R_0805_2012Metric"
 		(layer "F.Cu")
-		(at 149.75 101.4125 90)
+		(at 149.75 100.25 90)
 		(descr "Resistor SMD 0805 (2012 Metric), square (rectangular) end terminal, IPC_7351 nominal, (Body size source: IPC-SM-782 page 72, https://www.pcb-3d.com/wordpress/wp-content/uploads/ipc-sm-782a_amendment_1_and_2.pdf), generated with kicad-footprint-generator")
 		(tags "resistor")
@@
 	(footprint "Resistor_SMD:R_0805_2012Metric"
 		(layer "F.Cu")
-		(at 171.95 101.6625 90)
+		(at 171.95 100.275 90)
 		(descr "Resistor SMD 0805 (2012 Metric), square (rectangular) end terminal, IPC-7351 nominal, (Body size source: IPC-SM-782 page 72, https://www.pcb-3d.com/wordpress/wp-content/uploads/ipc-sm-782a_amendment_1_and_2.pdf), generated with kicad-footprint-generator")
 		(tags "resistor")
