File: TARA_T8X/TARA_T8X.kicad_pcb (KiCad board)
At the start: 2 copper layers, 122.5 x 87.9 mm, 125 parts, among them J1 Screw_Terminal_01x10, J2 ESP32-WROOM-32U, J3 Conn_01x04_MountingPin, J4 Screw_Terminal_01x10, Q1 2N5401, Q10 2N5401, Q2 2N5401, Q3 2N5401, Q4 2N5401, Q5 2N5401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

Commit message: 202510100506_greensave
Parts:
- U3: footprint my_footprint:RS485-TTL -> rs485_module:RS485-TTL
- moved C3 12.2 mm to (127.5, 63.5), turned to 0 degrees
- moved C2 7.01 mm to (113.4, 64.7), turned to 180 degrees
- moved U3 1.61 mm to (164.5, 85.1)
- moved RF1 0.66 mm to (137.0, 64.3)
- moved RF2 0.65 mm to (142.0, 64.4)
- moved C5 0.10 mm to (123.1, 63.5)
Routing:
- net /A: track 62.9 -> 9.73 mm
- net /B: track 57.2 -> 9.76 mm
- net /GPIO16: track 43.0 -> 0.00 mm, vias 3 -> 0
- net /GPIO17: track 39.7 -> 0.00 mm, vias 3 -> 0
- net Net-(J2-SENSOR_VN): track 87.2 -> 73.1 mm, vias 3 -> 2
- net /3V3: track 324.2 -> 319.2 mm, vias 11 -> 9
- net Net-(J2-IO33): track 93.6 -> 89.2 mm
- net /5V: track 130.6 -> 134.7 mm
- net /VCC: track 258.4 -> 255.5 mm, vias 12 -> 9
- net Net-(J2-IO5): track 49.4 -> 47.5 mm
- net Net-(J2-IO21): track 108.9 -> 107.2 mm
- net /BOOT: track 21.5 -> 23.1 mm
- net Net-(J2-SENSOR_VP): track 133.9 -> 132.9 mm
- net Net-(Q7-B): track 15.2 -> 14.5 mm
- net Net-(J2-IO34): track 120.1 -> 120.6 mm
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
Commit message: 202510110303_TARA_win10_kicad9
Parts:
- moved R18 1.50 mm to (160.8, 106.1)
- moved R20 1.04 mm to (175.8, 106.2)
- moved R19 0.59 mm to (168.4, 106.2)
Routing:
- net /A: track 9.73 -> 60.8 mm
- net /B: track 9.76 -> 58.6 mm
- net /GPIO17: track 0.00 -> 37.3 mm, vias 0 -> 3
- net /GPIO16: track 0.00 -> 33.9 mm, vias 0 -> 5
- net /VCC: track 255.5 -> 244.2 mm, vias 9 -> 10
- net Net-(D1-K): track 56.6 -> 49.9 mm
- net Net-(J2-IO27): track 67.6 -> 63.1 mm
- net Net-(J2-IO34): track 120.6 -> 116.6 mm
- net Net-(J2-IO25): track 83.8 -> 79.9 mm
- net Net-(J2-IO12): track 50.1 -> 47.1 mm, vias 3 -> 2
- net Net-(J2-IO19): track 39.7 -> 37.0 mm, vias 5 -> 4
- net Net-(J2-SENSOR_VN): track 73.1 -> 75.8 mm, vias 2 -> 1
- net Net-(J2-IO32): track 83.3 -> 80.9 mm
- net Net-(Q10-B): track 19.0 -> 17.3 mm
- net Net-(J2-IO23): track 41.9 -> 43.6 mm, vias 4 -> 2
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
Commit message: 202510110414_tara_win10_kicad9
Routing:
- net Net-(J2-IO34): track 116.6 -> 110.2 mm
- net Net-(J2-SENSOR_VN): track 75.8 -> 81.7 mm
- net Net-(J2-IO35): track 98.6 -> 92.8 mm
- net Net-(J2-SENSOR_VP): track 132.4 -> 126.7 mm
- net Net-(J2-IO22): track 118.3 -> 123.9 mm, vias 3 -> 2
- net /B: track 58.6 -> 54.9 mm
- net Net-(J4-Pin_2): track 19.8 -> 16.4 mm
- net Net-(J4-Pin_5): track 79.6 -> 82.1 mm
- net /3V3: track 319.1 -> 321.4 mm
- net Net-(J4-Pin_3): track 19.0 -> 16.8 mm, vias 2 -> 1
- net Net-(J4-Pin_1): track 15.2 -> 16.0 mm

Commit message: 202510131718_TARA_linux
Parts:
- moved R16 11.3 mm to (138.6, 102.2), turned to 180 degrees
- moved R14 11.1 mm to (123.6, 102.2), turned to 180 degrees
- moved R13 11.1 mm to (116.2, 102.2), turned to 180 degrees
- moved R15 11.0 mm to (131.2, 102.2), turned to 180 degrees
- moved J1 8.55 mm to (116.2, 128.5)
- moved Q1 8.28 mm to (106.7, 121.4)
- moved Q2 8.21 mm to (111.2, 121.5)
- moved R_led1 8.13 mm to (169.2, 124.4)
- moved R_led2 8.13 mm to (175.3, 124.4)
- moved RL1 8.13 mm to (159.0, 61.4)
- moved RL2 8.13 mm to (153.9, 61.4)
- moved BT1 8.13 mm to (188.2, 107.8)
- moved C3 8.13 mm to (116.0, 63.6)
- moved C4 8.13 mm to (80.5, 108.7)
- moved C4 8.13 mm to (116.0, 66.7)
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Routing:
- net /3V3: track 321.4 -> 302.1 mm, vias 9 -> 10
- net Net-(Q4-B): track 25.2 -> 12.0 mm
- net Net-(J2-IO22): track 123.9 -> 131.1 mm
- net Net-(D2-K): track 49.9 -> 53.1 mm
- net Net-(Q6-B): track 25.2 -> 22.3 mm
- net Net-(Q5-B): track 14.6 -> 12.1 mm
- net /GPIO16: track 33.9 -> 36.1 mm
- net /GPIO17: track 37.1 -> 39.2 mm
- net Net-(D3-K): track 78.9 -> 76.8 mm
- net Net-(Q3-B): track 11.6 -> 9.50 mm
- net Net-(Q1-B): track 48.4 -> 46.3 mm
- net /B: track 54.9 -> 53.1 mm
- net /A: track 60.4 -> 59.0 mm
- net Net-(Q2-B): track 23.8 -> 22.6 mm
- net /VCC: track 244.2 -> 245.5 mm
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
Commit message: 202510161151_Greensave_linux
Parts:
- removed R39: 560, Resistor_SMD:R_0805_2012Metric
- added R61: 560, Resistor_SMD:R_0805_2012Metric, F.Cu at (119.8, 77.7)
- added R62: 560, Resistor_SMD:R_0805_2012Metric, F.Cu at (109.7, 84.2)
- added R63: 560, Resistor_SMD:R_0805_2012Metric, F.Cu at (120.0, 97.7)
- added R64: 560, Resistor_SMD:R_0805_2012Metric, F.Cu at (127.2, 97.7)
- added R65: 560, Resistor_SMD:R_0805_2012Metric, F.Cu at (142.8, 82.8)
- added R66: 560, Resistor_SMD:R_0805_2012Metric, F.Cu at (142.5, 97.6)
- added R67: 560, Resistor_SMD:R_0805_2012Metric, F.Cu at (149.7, 97.5)
- added R68: 560, Resistor_SMD:R_0805_2012Metric, F.Cu at (153.5, 83.7)
- added R69: 560, Resistor_SMD:R_0805_2012Metric, F.Cu at (164.9, 83.7)
- added R70: 560, Resistor_SMD:R_0805_2012Metric, F.Cu at (172.7, 97.5)
- moved C4 119.1 mm to (186.3, 54.0)
- moved C5 23.1 mm to (99.0, 69.5), turned to 180 degrees
- moved R21 8.38 mm to (119.8, 72.7)
- moved R12 7.07 mm to (108.5, 102.2), turned to 180 degrees
- moved CR1 5.65 mm to (181.4, 57.0)
- moved Rbo1 5.65 mm to (181.4, 54.0)
- moved R23 2.41 mm to (120.0, 93.0)
- moved R24 2.37 mm to (127.2, 92.9)
- moved D1 1.64 mm to (97.0, 101.2)
- moved D2 1.50 mm to (97.0, 104.5)
- moved R11 1.42 mm to (111.0, 81.0)
- moved R22 1.38 mm to (112.2, 89.2)
- moved D3 1.36 mm to (97.0, 107.7)
- moved D4 1.23 mm to (97.0, 111.0)
- moved D5 1.03 mm to (97.0, 114.2)
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Routing:
- net GND: track 30.7 -> 43.5 mm, vias 68 -> 119
- net Net-(J2-IO12): track 47.1 -> 59.4 mm, vias 2 -> 4
- net Net-(J2-IO14): track 53.9 -> 66.2 mm, vias 2 -> 4
- net Net-(J2-IO32): track 81.2 -> 93.0 mm
- net Net-(J2-IO25): track 79.9 -> 91.2 mm
- net Net-(J2-IO26): track 73.5 -> 83.9 mm
- net /IO04: track 15.3 -> 21.7 mm
- net Net-(J2-IO21): track 108.3 -> 102.1 mm
- net Net-(OPTO1-Pad1): track 9.45 -> 3.32 mm
- net /EN: track 14.0 -> 19.0 mm
- net /5V: track 134.7 -> 139.4 mm
- net /3V3: track 302.1 -> 306.8 mm, vias 10 -> 8
- net Net-(J2-IO34): track 110.2 -> 106.4 mm
- net Net-(J4-Pin_5): track 82.1 -> 78.6 mm
- net Net-(J2-IO27): track 63.1 -> 66.3 mm
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
Commit message: 202510161400_greensave_win10
Routing:
- net Net-(J2-SENSOR_VN): track 80.8 -> 80.1 mm
- net /3V3: track 306.8 -> 306.1 mm
- net GND: vias 119 -> 121
Other:
- board text added: "202510161352"

Commit message: [200~20251016_G1730L
Routing:
- net Net-(Q8-B): track 17.3 -> 16.2 mm
Other:
- board text added: "20251016_G1715L"
- board text removed: "202510161352"

Commit message: 20251016_G1730L
Other:
- board text added: "20251016_G1730L"
- board text removed: "20251016_G1715L"
Changed lines of the file:
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@@
 		)
 	)
-	(gr_text "20251016_G1715L\n"
+	(gr_text "20251016_G1730L\n"
 		(at 184.8 124.25 0)
 		(layer "F.SilkS")
@@
 	)
 	(via
-		(at 180.75 124.95)
+		(at 180.741161 125.99989)
 		(size 0.8)
 		(drill 0.4)
@@
 	)
 	(via
-		(at 180.75 125.8)
+		(at 180.741136 127.249236)
 		(size 0.8)
 		(drill 0.4)
@@
 	)
 	(via
-		(at 180.75 123.25)
+		(at 180.741161 123.497053)
 		(size 0.8)
 		(drill 0.4)
@@
 	)
 	(via
-		(at 180.75 124.1)
+		(at 180.741161 124.748472)
 		(size 0.8)
 		(drill 0.4)
@@
 	)
 	(via
-		(at 180.75 122.4)
-		(size 0.8)
-		(drill 0.4)
+		(at 180.741161 122.245635)
+		(size 0.8)
+		(drill 0.4)
