File: TARA_T8X/TARA_T8X.kicad_pcb (KiCad board)
At the start: 2 copper layers, 122.5 x 87.9 mm, 134 parts, among them J1 Screw_Terminal_01x10, J2 ESP32-WROOM-32U, J3 Conn_01x04_MountingPin, J4 Screw_Terminal_01x10, Q1 2N5401, Q10 2N5401, Q2 2N5401, Q3 2N5401, Q4 2N5401, Q5 2N5401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

Commit message: 20251017_A0615W
Parts:
- moved R11 1.74 mm to (109.7, 79.8), turned to 0 degrees
- moved R68 1.01 mm to (153.8, 82.8)
- moved R69 0.98 mm to (164.9, 82.8)
Routing:
- net Net-(OPTO1-Pad4): track 7.87 -> 8.47 mm
Other:
- board text added: "20251017_A0615W"
- board text removed: "20251016_G1730L"
Changed lines of the file:
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@@
 	(footprint "Resistor_SMD:R_0805_2012Metric"
 		(layer "F.Cu")
-		(at 153.489488 83.730264 180)
+		(at 153.75 82.75 180)
 		(descr "Resistor SMD 0805 (2012 Metric), square (rectangular) end terminal, IPC-7351 nominal, (Body size source: IPC-SM-782 page 72, https://www.pcb-3d.com/wordpress/wp-content/uploads/ipc-sm-782a_amendment_1_and_2.pdf), generated with kicad-footprint-generator")
 		(tags "resistor")
@@
 	(footprint "Resistor_SMD:R_0805_2012Metric"
 		(layer "F.Cu")
-		(at 164.895164 83.733137 180)
+		(at 164.895164 82.75 180)
 		(descr "Resistor SMD 0805 (2012 Metric), square (rectangular) end terminal, IPC-7351 nominal, (Body size source: IPC-SM-782 page 72, https://www.pcb-3d.com/wordpress/wp-content/uploads/ipc-sm-782a_amendment_1_and_2.pdf), generated with kicad-footprint-generator")
 		(tags "resistor")
@@
 	(footprint "Resistor_SMD:R_0805_2012Metric"
 		(layer "F.Cu")
-		(at 110.980296 80.986896 90)
+		(at 109.749999 79.75)
 		(descr "Resistor SMD 0805 (2012 Metric), square (rectangular) end terminal, IPC-7351 nominal, (Body size source: IPC-SM-782 page 72, https://www.pcb-3d.com/wordpress/wp-content/uploads/ipc-sm-782a_amendment_1_and_2.pdf), generated with kicad-footprint-generator")
 		(tags "resistor")
 		(property "Reference" "R11"
-			(at 2.736896 0.019704 180)
+			(at 0 -2 180)
 			(layer "F.SilkS")
 			(effects
@@
 		)
 		(property "Value" "560"
-			(at 0 1.65 90)
+			(at 0 1.65 0)
 			(layer "F.Fab")
 			(hide yes)
@@
 		)
 		(property "Datasheet" "~"
-			(at 0 0 90)
+			(at 0 0 0)
 			(layer "F.Fab")
 			(hide yes)
@@
 		)
 		(property "Description" ""
-			(at 0 0 90)
+			(at 0 0 0)
 			(layer "F.Fab")
 			(hide yes)
@@
 		)
 		(fp_line
-			(start 1.68 -0.95)
-			(end 1.68 0.95)
+			(start -1.68 -0.95)
+			(end 1.68 -0.95)
 			(stroke
 				(width 0.05)
@@
 		)
 		(fp_line
-			(start -1.68 -0.95)
-			(end 1.68 -0.95)
+			(start -1.68 0.95)
+			(end -1.68 -0.95)
 			(stroke
 				(width 0.05)
@@
 		)
 		(fp_line
-			(start 1.68 0.95)
-			(end -1.68 0.95)
+			(start 1.68 -0.95)
+			(end 1.68 0.95)
 			(stroke
 				(width 0.05)
@@
 		)
 		(fp_line
-			(start -1.68 0.95)
-			(end -1.68 -0.95)
+			(start 1.68 0.95)
+			(end -1.68 0.95)
 			(stroke
 				(width 0.05)
@@
 		)
 		(fp_line
-			(start 1 -0.625)
-			(end 1 0.625)
+			(start -1 -0.625)
+			(end 1 -0.625)
 			(stroke
 				(width 0.1)
@@
 		)
 		(fp_line
-			(start -1 -0.625)
-			(end 1 -0.625)
+			(start -1 0.625)
+			(end -1 -0.625)
 			(stroke
 				(width 0.1)
@@
 		)
 		(fp_line
-			(start 1 0.625)
-			(end -1 0.625)
+			(start 1 -0.625)
+			(end 1 0.625)
 			(stroke
 				(width 0.1)
@@
 		)
 		(fp_line
-			(start -1 0.625)
-			(end -1 -0.625)
+			(start 1 0.625)
+			(end -1 0.625)
 			(stroke
 				(width 0.1)
@@
 		)
 		(fp_text user "${REFERENCE}"
-			(at 0 0 90)
+			(at 0 0 0)
 			(layer "F.Fab")
 			(effects
@@
 		)
 		(pad "1" smd roundrect
-			(at -0.9125 0 90)
+			(at -0.9125 0)
 			(size 1.025 1.4)
 			(layers "F.Cu" "F.Mask" "F.Paste")
@@
 		)
 		(pad "2" smd roundrect
-			(at 0.9125 0 90)
+			(at 0.9125 0)
 			(size 1.025 1.4)
 			(layers "F.Cu" "F.Mask" "F.Paste")
@@
 		)
 	)
-	(gr_text "20251016_G1730L\n"
+	(gr_text "20251017_A0615W\n"
 		(at 184.8 124.25 0)
 		(layer "F.SilkS")
@@
 	)
 	(segment
-		(start 110.980296 80.074396)
-		(end 116.824396 80.074396)
+		(start 117.37 80.37)
+		(end 117.37 81.875)
 		(width 0.4)
 		(layer "F.Cu")
@@
 	)
 	(segment
-		(start 117.37 80.62)
-		(end 117.37 81.875)
+		(start 110.662499 79.75)
+		(end 116.75 79.75)
 		(width 0.4)
 		(layer "F.Cu")
@@
 	)
 	(segment
-		(start 116.824396 80.074396)
-		(end 117.37 80.62)
+		(start 116.75 79.75)
+		(end 117.37 80.37)
 		(width 0.4)
 		(layer "F.Cu")
@@
 	)
 	(segment
+		(start 154.6625 82.75)
+		(end 157.5 82.75)
+		(width 0.4)
+		(layer "F.Cu")
+		(net 64)
+	)
+	(segment
 		(start 163.195 69.33)
 		(end 172.75 69.33)
@@
 	)
 	(segment
-		(start 154.401988 83.730264)
-		(end 157.480264 83.730264)
-		(width 0.4)
-		(layer "F.Cu")
-		(net 64)
-	)
-	(segment
 		(start 162.45 71.225)
 		(end 162.45 70.075)
@@
 	)
 	(segment
+		(start 157.5 82.75)
+		(end 157.5 80.215)
+		(width 0.4)
+		(layer "F.Cu")
+		(net 64)
+	)
+	(segment
 		(start 157.5 80.215)
 		(end 157.35 80.065)
@@
 	(segment
 		(start 157.5 83.75)
-		(end 157.5 80.215)
+		(end 157.5 82.75)
 		(width 0.4)
 		(layer "F.Cu")
@@
 	)
 	(segment
+		(start 106.75 79.75)
+		(end 105.65 80.85)
+		(width 0.4)
+		(layer "F.Cu")
+		(net 97)
+	)
+	(segment
 		(start 107.1 116.575)
 		(end 105.9 116.575)
@@
 	)
 	(segment
-		(start 106.575604 81.899396)
-		(end 110.980296 81.899396)
+		(start 105.65 80.85)
+		(end 105.65 83)
 		(width 0.4)
 		(layer "F.Cu")
@@
 	)
 	(segment
-		(start 105.9 116.575)
-		(end 105.65 116.325)
+		(start 105.65 83)
+		(end 105.65 82.825)
 		(width 0.4)
 		(layer "F.Cu")
@@
 	)
 	(segment
-		(start 107.645598 117.120598)
-		(end 107.1 116.575)
+		(start 108.837499 79.75)
+		(end 106.75 79.75)
 		(width 0.4)
 		(layer "F.Cu")
@@
 	)
 	(segment
-		(start 105.65 82.825)
-		(end 106.575604 81.899396)
+		(start 105.9 116.575)
+		(end 105.65 116.325)
+		(width 0.4)
+		(layer "F.Cu")
+		(net 97)
+	)
+	(segment
+		(start 107.645598 117.120598)
+		(end 107.1 116.575)
 		(width 0.4)
 		(layer "F.Cu")
@@
 	(segment
 		(start 105.65 116.325)
-		(end 105.65 82.825)
+		(end 105.65 83)
 		(width 0.4)
 		(layer "F.Cu")

Commit message: 20251016_G1700L
Parts:
- removed the C3 at (120.3, 59.6)
- removed the C3 at (116.0, 63.6)
- added C3: 10uf/50v, Capacitor_SMD:C_0805_2012Metric, F.Cu at (116.0, 63.3)
- moved R66 15.4 mm to (146.4, 82.8), turned to 0 degrees
- moved R67 15.2 mm to (153.5, 82.7), turned to 0 degrees
- moved R63 15.0 mm to (121.3, 82.7), turned to 0 degrees
- moved R64 15.0 mm to (127.6, 82.7), turned to 0 degrees
- moved Y1 14.8 mm to (131.2, 70.0), turned to 0 degrees
- moved R23 8.41 mm to (116.1, 85.5), turned to 180 degrees
- moved R24 8.23 mm to (123.6, 85.5), turned to 0 degrees
- moved RF1 7.83 mm to (122.1, 59.7)
- moved RF2 7.48 mm to (127.4, 59.7)
- moved R30 7.46 mm to (167.7, 85.5), turned to 0 degrees
- moved R29 6.84 mm to (160.3, 85.5), turned to 180 degrees
- moved R28 6.51 mm to (153.5, 85.5), turned to 0 degrees
- moved R68 6.49 mm to (160.2, 82.7)
- moved R27 6.45 mm to (146.1, 85.5), turned to 0 degrees
- moved R26 6.44 mm to (138.7, 85.5), turned to 180 degrees
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Connections:
- Y1 pad 1: Net-(U4-X1) -> Net-(U4-X2)
- Y1 pad 2: Net-(U4-X2) -> Net-(U4-X1)
Routing:
- net Net-(J2-IO15): track 18.5 -> 31.4 mm
- net Net-(J2-IO22): track 130.8 -> 118.1 mm
- net Net-(U4-X1): track 10.00 -> 22.5 mm
- net Net-(J2-IO14): track 66.2 -> 53.9 mm, vias 4 -> 2
- net Net-(U4-X2): track 5.22 -> 17.2 mm
- net Net-(J2-IO12): track 59.4 -> 47.5 mm, vias 4 -> 2
- net Net-(J2-IO26): track 83.9 -> 72.9 mm
- net Net-(OPTO4-Pad1): track 7.29 -> 13.9 mm, vias 0 -> 2
- net /A: track 59.0 -> 65.5 mm
- net /B: track 53.1 -> 59.2 mm
- net Net-(J2-IO25): track 91.4 -> 85.3 mm, vias 2 -> 6
- net /3V3: track 306.1 -> 300.2 mm
- net Net-(J2-IO32): track 93.0 -> 87.7 mm
- net Net-(J2-IO33): track 89.6 -> 94.9 mm, vias 2 -> 5
- net Net-(J2-IO2): track 62.3 -> 59.5 mm
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Other:
- board text added: "20251017_G1645L"
- board text removed: "20251017_A0615W"

Commit message: Update TARA_T8X.kicad_pcb
Parts:
- moved R21 1.09 mm to (120.8, 72.8), turned to 0 degrees
- moved R61 1.00 mm to (120.8, 77.7), turned to 180 degrees
Routing:
- net Net-(OPTO4-Pad1): track 13.9 -> 15.7 mm
- net Net-(J2-IO32): track 87.7 -> 86.7 mm
- net GND: vias 116 -> 118
Other:
- board text added: "20251018_A0649W"
- board text removed: "20251017_G1645L"

Commit message: 20251018_1500TL
Parts:
- moved R63 2.30 mm to (123.6, 82.8)
- moved R30 1.11 mm to (168.8, 85.5)
- moved R22 1.07 mm to (108.6, 85.5)
- moved R11 1.03 mm to (108.7, 79.7)
- moved R62 1.03 mm to (108.7, 82.7)
- moved R29 0.96 mm to (161.3, 85.4)
- moved R66 0.32 mm to (146.1, 82.7)
- moved R26 0.26 mm to (139.0, 85.5)
- moved R7 0.22 mm to (146.4, 119.9)
- moved R6 0.21 mm to (141.3, 119.9)
- moved R4 0.20 mm to (131.2, 119.9)
- moved R3 0.19 mm to (125.9, 119.9)
- moved R2 0.17 mm to (120.4, 120.0)
- moved R1 0.16 mm to (115.9, 120.0)
- moved R38 0.10 mm to (159.2, 64.1)
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Routing:
- net /IO04: track 19.5 -> 23.7 mm, vias 2 -> 3
- net Net-(J2-IO19): track 37.0 -> 39.5 mm
- net Net-(J2-IO25): track 85.3 -> 87.5 mm
- net /A: track 65.5 -> 67.6 mm
- net GND: track 43.5 -> 45.3 mm, vias 118 -> 128
- net Net-(J2-IO33): track 94.9 -> 96.5 mm, vias 5 -> 4
- net Net-(OPTO10-Pad1): track 6.17 -> 5.05 mm
- net Net-(OPTO1-Pad4): track 8.47 -> 9.51 mm
- net Net-(OPTO2-Pad1): track 3.85 -> 4.85 mm
- net Net-(J2-IO15): track 31.4 -> 32.4 mm
- net Net-(Q1-B): track 45.0 -> 44.2 mm
- net Net-(OPTO9-Pad1): track 4.04 -> 3.40 mm
- net Net-(J2-IO5): track 46.1 -> 45.5 mm
Other:
- board text added: "20251018_1200TL"
- board text removed: "20251018_A0649W"

Commit message: 20251018_1515TL_FINAL
Routing:
- net GND: track 45.3 -> 51.3 mm
- net Net-(J2-IO5): track 45.5 -> 44.0 mm
Other:
- board text added: "20251018_1515TL_FINAL"
- board text removed: "20251018_1200TL"

Commit message: 20251022_T1538L
Parts:
- moved C5 0.88 mm to (116.0, 58.7)
Routing:
- net GND: vias 128 -> 130
Changed lines of the file:
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@@
 		)
 		(embedded_fonts no)
-		(model "/home/boon/Downloads/ESP32-WROOM-32UE.wrl"
+		(model "/home/boon/Downloads/ESP32-S2-WROOM.wrl"
 			(offset
 				(xyz 0 0 0)
@@
 		(tags "capacitor")
 		(property "Reference" "C4"
-			(at -2.95 0 0)
+			(at -2.519034 0.007329 0)
 			(layer "F.SilkS")
 			(effects
@@
 	(footprint "Capacitor_SMD:C_0805_2012Metric"
 		(layer "F.Cu")
-		(at 115.98 59.605)
+		(at 115.969999 58.725857)
 		(descr "Capacitor SMD 0805 (2012 Metric), square (rectangular) end terminal, IPC_7351 nominal, (Body size source: IPC-SM-782 page 76, https://www.pcb-3d.com/wordpress/wp-content/uploads/ipc-sm-782a_amendment_1_and_2.pdf, https://docs.google.com/spreadsheets/d/1BsfQQcO9C6DZCsRaXUlFlo91Tg2WpOkGARC1WS5S8t0/edit?usp=sharing), generated with kicad-footprint-generator")
 		(tags "capacitor")
@@
 		)
 	)
-	(gr_text " SCL\n (A) "
+	(gr_text " SCL\n  (A) "
 		(at 128.591101 55.947446 0)
 		(layer "F.SilkS")
@@
 	)
 	(via
+		(at 120.64 66.88)
+		(size 0.8)
+		(drill 0.4)
+		(layers "F.Cu" "B.Cu")
+		(free yes)
+		(net 1)
+	)
+	(via
 		(at 160 87)
 		(size 0.8)
@@
 	)
 	(via
+		(at 111.72 62.41)
+		(size 0.8)
+		(drill 0.4)
+		(layers "F.Cu" "B.Cu")
+		(free yes)
+		(net 1)
+	)
+	(via
 		(at 172.75 56.25)
 		(size 0.8)
@@
 	)
 	(via
-		(at 116.75 63.55)
+		(at 118.49 63.83)
 		(size 0.8)
 		(drill 0.4)
@@
 	)
 	(segment
-		(start 112.07 60.845)
-		(end 112.06 60.835)
-		(width 0.6)
-		(layer "F.Cu")
-		(net 9)
-	)
-	(segment
 		(start 79.475 86.175)
 		(end 79.45 86.15)
@@
 	)
 	(segment
+		(start 115.019999 58.725857)
+		(end 113.809143 58.725857)
+		(width 0.6)
+		(layer "F.Cu")
+		(net 9)
+	)
+	(segment
 		(start 79.45 86.15)
 		(end 79.45 102.375)
@@
 	)
 	(segment
-		(start 112.06 60.835)
+		(start 113.809143 58.725857)
+		(end 111.7 60.835)
+		(width 0.6)
+		(layer "F.Cu")
+		(net 9)
+	)
+	(segment
+		(start 111.7 60.835)
 		(end 107.19 60.835)
 		(width 0.6)
@@
 		(width 0.6)
 		(layer "F.Cu")
-		(net 9)
-	)
-	(segment
-		(start 112.07 60.845)
-		(end 113.31 59.605)
-		(width 0.6)
-		(layer "F.Cu")
-		(net 9)
-	)
-	(segment
-		(start 115.03 59.605)
-		(end 113.31 59.605)
-		(width 0.6)
-		(layer "F.Cu")
