File: TARA_T8X/TARA_T8X.kicad_sch (KiCad schematic)
At the start: 120 parts, among them J1 Screw_Terminal_01x10, J2 ESP32-WROOM-32U, J3 Conn_01x04_MountingPin, J4 Screw_Terminal_01x10, Q1 2N5401, Q10 2N5401, Q2 2N5401, Q3 2N5401, Q4 2N5401, Q5 2N5401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

Commit message: 202510100506_greensave
Parts:
- U3: footprint my_footprint:RS485-TTL -> rs485_module:RS485-TTL
Changed lines of the file:
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@@
 	(wire
 		(pts
+			(xy 182.88 224.79) (xy 219.71 224.79)
+		)
+		(stroke
+			(width 0)
+			(type default)
+		)
+	)
+	(wire
+		(pts
 			(xy 113.03 199.39) (xy 111.76 198.12)
 		)
@@
 			)
 		)
-		(property "Footprint" "my_footprint:RS485-TTL"
+		(property "Footprint" "rs485_module:RS485-TTL"
 			(at 234.823 177.8 0)
 			(effects

Commit message: 202510161151_Greensave_linux
Parts:
- added R61, R62, R63, R64, R65, R66, R67, R68, R69, R70: 560, Resistor_SMD:R_0805_2012Metric, symbol Device:R_Small
Connections:
- net GND: now also R61.2, R62.2, R63.2, R64.2, R65.2, R66.2, R67.2, R68.2, R69.2, R70.2
- net IO04: now also R70.1
- net at J2.23 (IO15), R29.2: now also R69.1
- net at J2.13 (IO14), R26.1: now also R66.1
- net at J2.14 (IO12), R27.2: now also R67.1
- net at J2.9 (IO33), R22.2: now also R62.1
- net at J2.16 (IO13), R28.2: now also R68.1
- net at J2.10 (IO25), R23.1: now also R63.1
- net at J2.11 (IO26), R24.2: now also R64.1
- net at J2.12 (IO27), R25.2: now also R65.1
- net at J2.8 (IO32), R21.2: now also R61.1

Commit message: 20251016_G1700L
Connections:
- net at U4.1 (X1): now also Y1.2; no longer Y1.1
- net at U4.2 (X2): now also Y1.1; no longer Y1.2
Other:
- moved on the sheet: BT1, C1, C2, C3, C4, C5, CR1, D1, D10, D2, D3, D4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
